File: src/LEDMemoryGame.kicad_pcb (KiCad board)
At the start: 2 copper layers, 69.1 x 53.9 mm, 15 parts, among them SW1 RED, SW2 BLUE, SW3 YELLOW, SW4 GREEN

Commit message: Update repo
Updated all the files to make the PCB Better
Parts:
- added G***: LOGO, LOGO, F.Cu at (127.4, 120.6)
- added G***: LOGO, LOGO, B.Cu at (130.1, 119.2)
- added G***: LOGO, LOGO, B.Cu at (120.5, 121.3)
- added G***: LOGO, LOGO, B.Cu at (123.0, 128.0)
- added G***: LOGO, LOGO, F.Cu at (145.9, 116.6)
- added G***: LOGO, LOGO, F.Cu at (162.3, 115.6)
- added G***: LOGO, LOGO, F.Cu at (141.0, 91.2)
- added G***: LOGO, LOGO, F.Cu at (144.1, 125.5)
- added G***: LOGO, LOGO, F.Cu at (122.7, 101.7)
- added G***: LOGO, LOGO, B.Cu at (122.5, 116.7)
- added G***: LOGO, LOGO, B.Cu at (152.8, 116.5)
- added G***: LOGO, LOGO, B.Cu at (123.3, 95.3)
- moved BT1 41.7 mm to (172.8, 114.4)
- moved R3 41.7 mm to (164.6, 86.6)
- moved R4 41.7 mm to (178.3, 86.6)
- moved A1 41.7 mm to (117.6, 131.2)
- moved BZ1 41.7 mm to (120.9, 84.4)
- moved D1 41.7 mm to (130.8, 90.2)
- moved D4 41.7 mm to (172.2, 90.2)
- moved R1 41.7 mm to (137.1, 86.6)
- moved R2 41.7 mm to (150.9, 86.6)
- moved SW2 41.7 mm to (142.0, 101.0)
- moved SW3 41.7 mm to (155.6, 101.0)
- moved D2 41.7 mm to (144.6, 90.2)
- moved D3 41.7 mm to (158.4, 90.2)
- moved SW1 41.7 mm to (128.3, 101.0)
- moved SW4 41.7 mm to (169.3, 101.0)
Routing:
- net GND: track 169.4 -> 136.5 mm
Other:
- board size 69.1 x 53.9 mm -> 69.1 x 53.8 mm
